File: samples/iot_sensor_node/iot_sensor_node.kicad_sch (KiCad schematic)
At the start: 21 parts, among them J1 USB-C, U1 AP62300, U2 TLV75518, U3 ESP32-WROOM-32E, U4 BME280

Commit message: chore: regenerate 8 sample designs against v0.27.0 engine
All 8 samples pass full validation (0 ERC errors):
- led_power_indicator, iot_sensor_node, usb_regulated_supply,
  usb_uart_bridge, oled_display_module, battery_iot_sensor,
  motor_controller, fpga_power_carrier

New artifacts per sample: .kicad_sch, _test_points.csv, _pinout.csv,
canonical_spec.yaml, design_ir.json, validation_report.json; MCU samples
also emit sdkconfig.defaults / .ioc stubs.

Also adds samples/*/svg/ to .gitignore — schematic SVG exports are
regenerable and too large to track.

zigbee_humidistat deferred: non-deterministic schematic output across
two generation runs (text annotation ordering vs sheet_instances).
Parts:
- U4: footprint Package_LGA:Bosch_LGA-8_2.5x2.5mm_P0.65mm_ClockwisePinNumbering -> Package_LGA:Bosch_LGA-8_2.5x2.5mm
Connections:
- net VDD_1P8 is gone; now on net GND: C6.2, U2.5 (OUT)
- net ESP_EN: now also R5.2; no longer R5.1
- net GND: now also R1.2, R2.2, R5.1; no longer R1.1, R2.1, R5.2, R6.2, U3.25 (IO0)
- net VBUS_5V: now also J1.A5 (CC1), J1.B5 (CC2), R1.1, R2.1
- removed net USB_CC1: J1.A5 (CC1), R1.2
- removed net USB_CC2: J1.B5 (CC2), R2.2
- new net ESP_IO0: R6.2, U3.25 (IO0)
Other:
- note added: "TP1: GND [ground]"
- note added: "TP2: VBUS_5V [power_rail]"
- note added: "TP3: VDD_1P8 [power_rail]"
- note added: "TP4: VDD_3P3 [power_rail]"
- moved on the sheet: C1
