File: samples/usb_regulated_supply/usb_regulated_supply.kicad_sch (KiCad schematic)
At the start: 14 parts, among them J1 USB-C, U1 AP62300, U2 TLV75518

Commit message: chore: regenerate 8 sample designs against v0.27.0 engine
All 8 samples pass full validation (0 ERC errors):
- led_power_indicator, iot_sensor_node, usb_regulated_supply,
  usb_uart_bridge, oled_display_module, battery_iot_sensor,
  motor_controller, fpga_power_carrier

New artifacts per sample: .kicad_sch, _test_points.csv, _pinout.csv,
canonical_spec.yaml, design_ir.json, validation_report.json; MCU samples
also emit sdkconfig.defaults / .ioc stubs.

Also adds samples/*/svg/ to .gitignore — schematic SVG exports are
regenerable and too large to track.

zigbee_humidistat deferred: non-deterministic schematic output across
two generation runs (text annotation ordering vs sheet_instances).
Connections:
- net VDD_1P8 is gone; now on net GND: C6.2, U2.5 (OUT)
- net GND: now also R1.2, R2.2; no longer C3.2, C5.2, L1.2, R1.1, R2.1, R3.1, R3.2, R4.2, U1.4 (FB), U2.1 (IN), U2.3 (EN)
- net VBUS_5V: now also J1.A5 (CC1), J1.B5 (CC2), R1.1, R2.1
- removed net USB_CC1: J1.A5 (CC1), R1.2
- removed net USB_CC2: J1.B5 (CC2), R2.2
- new net VDD_3P3: C3.2, C5.2, L1.2, R3.1, R3.2, R4.2, U1.4 (FB), U2.1 (IN), U2.3 (EN)
Other:
- note added: "TP1: GND [ground]"
- note added: "TP2: VBUS_5V [power_rail]"
- note added: "TP3: VDD_1P8 [power_rail]"
- note added: "TP4: VDD_3P3 [power_rail]"
- moved on the sheet: C1
